File: keychain/ruddock_crest.kicad_pcb (KiCad board)
At the start: 2 copper layers, 76.1 x 83.8 mm, 3 parts

Commit message: Add silkscreen footprint on back
Parts:
- added G***: LOGO, crest:ruddock_fsilk_small, B.Cu at (142.2, 101.6)
